Commit message: limit pan joint to +/-180 deg

File: src/roarm/urdf/roarm.urdf (robot description, URDF)
Before this commit: robot physics, 11 links, 10 joints
Joints:
- joint base_to_L1: limit lower=-3.14 upper=3.14 effort=1000.0 velocity=0.5 -> lower=-1.5707 upper=1.5707 effort=1000.0 velocity=0.5

Commit message: adjust L2 angle to ensure 0 is vertical

File: src/roarm/urdf/roarm.urdf (robot description, URDF)
Before this commit: robot physics, 11 links, 10 joints
Joints:
- joint L1_to_L2: limit lower=-1.0467 upper=1.0467 effort=1000.0 velocity=0.5 -> lower=-1.8326 upper=0.2617 effort=1000.0 velocity=0.5; origin xyz=0 0.041051 0.0534 -> xyz=0 0.041051 0.0534 rpy=0.7854 0 0
